File: takshaka-mux-board.kicad_sch (KiCad schematic)
At the start: 8 parts, among them J1 Conn_01x01_Male, J2 Conn_01x01_Male, J3 Conn_02x08_Counter_Clockwise, J4 Conn_01x08_Male, U1 4051, U2 4051

Commit message: v0.2
Parts:
- removed J4: Conn_01x08_Male, Connector_PinHeader_2.54mm:PinHeader_1x08_P2.54mm_Vertical, symbol Connector:Conn_01x08_Male
- added J4: Conn_01x08_Female, Connector_PinSocket_2.54mm:PinSocket_1x08_P2.54mm_Vertical, symbol Connector:Conn_01x08_Female
- added J5, J6: Conn_01x01_Male, Connector_PinHeader_2.54mm:PinHeader_1x01_P2.54mm_Vertical, symbol Connector:Conn_01x01_Male
Connections:
- net +3V3_A: now also J4.1 (Pin_1)
- net CHANNEL_SELECT_A: now also J4.2 (Pin_2)
- net CHANNEL_SELECT_B: now also J4.3 (Pin_3)
- net CHANNEL_SELECT_C: now also J4.4 (Pin_4)
- net GND: now also J4.8 (Pin_8)
- net MUX_1_SIGNAL: now also J4.5 (Pin_5)
- net MUX_2_SIGNAL: now also J4.6 (Pin_6)
- net ATTACK renamed A
- net DECAY renamed D|R
- net DRIVE renamed D
- net P_D_MOD renamed PD_MOD
- net P_H_MOD renamed PH_MOD
- net P_S_MOD renamed PS_MOD
- net RES renamed R
- net RUMBLE renamed GROWL
- net SUSTAIN renamed S
- net S_C_MOD renamed SH_MOD
- net S_D_MOD renamed SD_MOD
- net S_S_MOD renamed SS_MOD
- no-connect marks 3 -> 5
Other:
- note added: "Daisy Seed I/O"
- note added: "Mounting Pins"
- note added: "Mux Inputs"
- moved on the sheet: C1, C2, J1, J2, J3, U1, U2

Commit message: added schematic PDF.
Other:
- company: (none) -> Song Naga
- title: (none) -> Simple Multiplexer
Changed lines of the file:
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@@
 (kicad_sch (version 20211123) (generator eeschema)
   (paper "A4")
+  (title_block
+    (title "Simple Multiplexer")
+    (date "2022-09-21")
+    (rev "v0.2")
+    (company "Song Naga")
+  )
   (junction (at 51.054 98.806) (diameter 0) (color 0 0 0 0)
   )
